File: SensorBoard/SensorBoard.sch (EAGLE design)
At the start: 21 parts, among them IC1 MEGA8-AI, IC2 SN65176D, IC3 LM2936M-3.3, IC4 LM2936M-5.0

Commit message: finished sensor board schematic
Parts:
- added C10, C11, C12, C13, C14, C15, C16, C8, C9: 100n, resistor:C-EUC0603
- added C6: 330n, resistor:C-EUC0603
- added C7: 56p, resistor:C-EUC0603
Connections:
- new net +3V3: C10.1, C14.1, C4.1, IC3.VO, R5.2, R6.2, U$1.NCS, U$1.RESV, U$1.VDD, U$1.VDDIO, U$2.P$1, U$3.P$1
- new net +5V: C13.1, C16.1, C3.1, C8.1, C9.1, IC1.AVCC, IC1.VCC@1, IC1.VCC@2, IC2.VCC, IC4.VO, JP2.3, R1.2, R2.2, R3.2, R4.2
- new net -RE: IC1.PD4(XCK/T0), IC2.!RE, R1.1
- new net DE: IC1.PD3(INT1), IC2.DE
- new net DTR: C15.1, JP2.6
- new net GND: C1.2, C10.2, C11.2, C12.2, C13.2, C14.2, C16.2, C2.2, C3.2, C4.2, C5.2, C6.2, C7.2, C8.2, C9.2, IC1.GND, IC1.GND@1, IC1.GND@2, IC2.GND, IC3.GND@1, IC3.GND@2, IC3.GND@3, IC3.GND@4, IC4.GND@1, IC4.GND@2, IC4.GND@3, IC4.GND@4, JP1.7, JP1.8, JP2.1, JP2.2, U$1.ADO/SDO, U$1.FSYNC, U$1.GND, U$1.PAD, U$1.RESV2
- new net INT: IC1.PD2(INT0), U$1.INT
- new net N$1: IC2.A, JP1.3, JP1.4
- new net N$2: IC2.B, JP1.5, JP1.6
- new net N$3: R6.1, U$1.SCL/SCLK, U$2.P$2
- new net N$4: C11.1, U$1.REGOUT
- new net N$5: C5.1, IC1.PB6(XTAL1/TOSC1), U$4.P$1
- new net N$6: R5.1, U$1.SDA/SDI, U$3.P$2
- new net N$7: C7.1, IC1.PB7(XTAL2/TOSC2), U$4.P$2
- new net N$8: C15.2, IC1.PC6(/RESET), R2.1
- new net N$9: C12.1, IC1.AREF
- new net RX: IC1.PD0(RXD), IC2.R, JP2.4
- new net SCL: IC1.PC5(ADC5/SCL), R3.1, U$2.P$3
- new net SDA: IC1.PC4(ADC4/SDA), R4.1, U$3.P$3
- new net TX: IC1.PD1(TXD), IC2.D, JP2.5
- new net VCC: C1.1, C2.1, C6.1, IC3.VIN, IC4.VIN, JP1.1, JP1.2
Other:
- moved on the sheet: C1, C2, C3, C4, C5, IC1, IC2, IC3, IC4, JP1, JP2, R1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

Commit message: finished sensor board layout
Parts:
- removed JP2: (no value), pinhead:PINHD-1X6
- added U$5: FTDI-PINHEADER, FTDI-PINHEADER:FTDI-PINHEADER
Connections:
- net +5V: now also U$5.VCC; no longer JP2.3
- net DTR: now also U$5.DTR; no longer JP2.6
- net GND: now also JP1.1, JP1.2, U$5.CTS, U$5.GND; no longer JP1.7, JP1.8, JP2.1, JP2.2
- net N$1: now also JP1.5, JP1.6; no longer JP1.3, JP1.4
- net N$2: now also JP1.3, JP1.4; no longer JP1.5, JP1.6
- net RX: now also U$5.TX; no longer JP2.4
- net TX: now also U$5.RX; no longer JP2.5
- net VCC: now also JP1.7, JP1.8; no longer JP1.1, JP1.2
Other:
- moved on the sheet: JP1
