File: SensorBoard/SensorBoard2.brd (EAGLE design)
At the start: 37.8 x 19.5 mm, 33 parts, among them IC1 MEGA8-AI, IC2 SN65176D, IC3 LM2936M-3.3, IC4 LM2936M-5.0

Commit message: added pads for flashing the bootloader to sensor board, added alternative version of sensor board
Parts:
- moved C16 5.18 mm to (9.65, 20.6)
- moved C2 5.18 mm to (2.29, 20.6)
- moved C11 5.18 mm to (34.1, 19.8)
- moved C7 5.18 mm to (11.4, 10.9)
- moved C8 5.18 mm to (18.3, 9.91)
- moved JP1 5.18 mm to (0.51, 13.0)
- moved C1 5.18 mm to (4.32, 19.6)
- moved C14 5.18 mm to (32.5, 12.4)
- moved C3 5.18 mm to (9.91, 14.0)
- moved C6 5.18 mm to (32.5, 7.62)
- moved C9 5.18 mm to (18.3, 12.2)
- moved IC2 5.18 mm to (12.7, 15.0)
- moved R1 5.18 mm to (15.5, 14.7)
- moved R4 5.18 mm to (23.9, 18.8)
- moved U$1 5.18 mm to (32.5, 17.5)
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Other:
- board size 37.8 x 19.5 mm -> 38.8 x 29.7 mm
